File: Actionneur_Gros_Robot.brd (EAGLE design)
At the start: 110 x 55 mm, 52 parts, among them M1 ARDUINO-NANO-3.0, M10 SERVO, M11 SERVO, M2 SERVO, M3 SERVO, M4 SERVO, M5 SERVO, M6 SERVO, M7 SERVO, M8 SERVO, M9 SERVO, Y1 16MHz

Commit message: revA2
Connections:
- net VCC: now also J3.17, J3.18; no longer J3.21, J3.22
- net VDD: now also J3.21, J3.22; no longer J3.17, J3.18
Routing:
- net VCC: track 217.4 -> 216.3 mm
- net CANL: track 72.1 -> 71.2 mm
- net VDD: track 275.0 -> 274.5 mm, vias 6 -> 7
Changed lines of the file:
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@@
 <contactref element="R13" pad="2"/>
 <contactref element="M1" pad="J2.4"/>
-<contactref element="J3" pad="22"/>
-<contactref element="J3" pad="21"/>
 <contactref element="SV4" pad="6"/>
 <contactref element="SV4" pad="4"/>
@@
 <wire x1="102.33" y1="22.74" x2="102.33" y2="20.2" width="0.1524" layer="1"/>
 <wire x1="102.33" y1="17.66" x2="102.33" y2="20.2" width="0.1524" layer="1"/>
-<wire x1="32.21" y1="49.27" x2="32.21" y2="51.81" width="0.1524" layer="1"/>
 <wire x1="65.02" y1="34.4" x2="61.1" y2="34.4" width="0.1524" layer="1"/>
 <wire x1="61.1" y1="34.4" x2="55.8" y2="29.1" width="0.1524" layer="1"/>
@@
 <wire x1="30.27" y1="46.77" x2="27.93" y2="46.77" width="0.1524" layer="1"/>
 <wire x1="27.93" y1="46.77" x2="27.87" y2="46.83" width="0.1524" layer="1"/>
-<wire x1="32.21" y1="49.27" x2="32.21" y2="47.71" width="0.1524" layer="1"/>
-<wire x1="31.27" y1="46.77" x2="30.27" y2="46.77" width="0.1524" layer="1"/>
-<wire x1="32.21" y1="47.71" x2="31.27" y2="46.77" width="0.1524" layer="1"/>
 <wire x1="27.87" y1="46.83" x2="25.83" y2="46.83" width="0.1524" layer="1"/>
 <wire x1="24.2" y1="45.2" x2="25.83" y2="46.83" width="0.1524" layer="1"/>
@@
 <wire x1="16.7" y1="38.5" x2="19.81480625" y2="38.5" width="0.1524" layer="1"/>
 <wire x1="24.2" y1="42.88519375" x2="24.2" y2="45.2" width="0.1524" layer="1"/>
+<contactref element="J3" pad="18"/>
+<contactref element="J3" pad="17"/>
+<wire x1="27.13" y1="49.27" x2="27.13" y2="51.81" width="0.1524" layer="1"/>
+<wire x1="27.87" y1="46.83" x2="27.87" y2="48.53" width="0.1524" layer="1"/>
+<wire x1="27.87" y1="48.53" x2="27.13" y2="49.27" width="0.1524" layer="1"/>
 </signal>
 <signal name="I2C_SDA">
@@
 <contactref element="R15" pad="2"/>
 <contactref element="R14" pad="2"/>
-<contactref element="J3" pad="18"/>
-<contactref element="J3" pad="17"/>
 <contactref element="LED3" pad="K"/>
 <contactref element="U$3" pad="18"/>
@@
 <wire x1="68.1" y1="50.5" x2="72.37" y2="50.5" width="0.1524" layer="1"/>
 <wire x1="72.37" y1="50.5" x2="72.67" y2="50.2" width="0.1524" layer="1"/>
-<wire x1="27.13" y1="49.27" x2="27.13" y2="51.81" width="0.1524" layer="1"/>
 <wire x1="76.17" y1="4.1" x2="77.7" y2="4.1" width="0.1524" layer="1"/>
 <wire x1="79.3" y1="2.5" x2="92.4" y2="2.5" width="0.1524" layer="1"/>
@@
 <wire x1="33.38" y1="34.07" x2="35.92" y2="34.07" width="0.1524" layer="1"/>
 <wire x1="50.1" y1="46.6" x2="42.2" y2="46.6" width="0.1524" layer="1"/>
-<wire x1="42.2" y1="46.6" x2="41.6" y2="46" width="0.1524" layer="1"/>
-<wire x1="41.6" y1="46" x2="41.6" y2="45.9" width="0.1524" layer="1"/>
-<via x="41.6" y="45.9" extent="1-16" drill="0.35"/>
-<wire x1="41.6" y1="45.9" x2="37.8" y2="42.1" width="0.1524" layer="16"/>
-<wire x1="37.8" y1="42.1" x2="37.8" y2="38.3" width="0.1524" layer="16"/>
+<wire x1="42.2" y1="46.6" x2="41.9" y2="46.3" width="0.1524" layer="1"/>
+<wire x1="41.9" y1="46.3" x2="41.2" y2="46.3" width="0.1524" layer="1"/>
 <via x="37.8" y="38.3" extent="1-16" drill="0.35"/>
 <wire x1="37.8" y1="38.3" x2="37.8" y2="34.7" width="0.1524" layer="1"/>
@@
 <wire x1="35.92" y1="34.07" x2="35.95" y2="34.1" width="0.1524" layer="1"/>
 <wire x1="50.1" y1="46.6" x2="51.04" y2="47.54" width="0.1524" layer="1"/>
-<wire x1="37.8" y1="42.1" x2="36.8" y2="43.1" width="0.1524" layer="16"/>
-<wire x1="36.8" y1="43.1" x2="36.8" y2="45.9" width="0.1524" layer="16"/>
-<wire x1="36.8" y1="45.9" x2="34.9" y2="47.8" width="0.1524" layer="16"/>
-<wire x1="27.7" y1="47.8" x2="27" y2="48.5" width="0.1524" layer="16"/>
-<wire x1="27" y1="48.5" x2="27" y2="49.14" width="0.1524" layer="16"/>
-<wire x1="27" y1="49.14" x2="27.13" y2="49.27" width="0.1524" layer="16"/>
-<wire x1="34.9" y1="47.8" x2="27.7" y2="47.8" width="0.1524" layer="16"/>
 <wire x1="5.92" y1="32.11" x2="5.92" y2="34.65" width="0.1524" layer="1"/>
 <wire x1="5.92" y1="29.57" x2="5.92" y2="32.11" width="0.1524" layer="1"/>
 <wire x1="17.57" y1="47.3" x2="5.92" y2="35.65" width="0.1524" layer="1"/>
 <wire x1="5.92" y1="34.65" x2="5.92" y2="35.65" width="0.1524" layer="1"/>
-<wire x1="25.7" y1="47.3" x2="27.13" y2="48.73" width="0.1524" layer="1"/>
-<wire x1="27.13" y1="48.73" x2="27.13" y2="49.27" width="0.1524" layer="1"/>
-<wire x1="17.57" y1="47.3" x2="25.7" y2="47.3" width="0.1524" layer="1"/>
+<wire x1="17.57" y1="47.3" x2="20.8" y2="47.3" width="0.1524" layer="1"/>
 <wire x1="51.04" y1="47.54" x2="65.14" y2="47.54" width="0.1524" layer="1"/>
 <wire x1="65.14" y1="47.54" x2="68.1" y2="50.5" width="0.1524" layer="1"/>
@@
 <wire x1="20.18" y1="40.6" x2="21.67" y2="42.09" width="0.1524" layer="1"/>
 <wire x1="12.3" y1="40.6" x2="20.18" y2="40.6" width="0.1524" layer="1"/>
+<contactref element="J3" pad="22"/>
+<contactref element="J3" pad="21"/>
+<wire x1="32.21" y1="49.27" x2="32.21" y2="51.81" width="0.1524" layer="1"/>
+<wire x1="20.8" y1="47.3" x2="21.3" y2="47.8" width="0.1524" layer="1"/>
+<via x="21.3" y="47.8" extent="1-16" drill="0.35"/>
+<wire x1="21.3" y1="47.8" x2="30.74" y2="47.8" width="0.1524" layer="16"/>
+<wire x1="30.74" y1="47.8" x2="32.21" y2="49.27" width="0.1524" layer="16"/>
+<wire x1="37.8" y1="38.3" x2="37.8" y2="42.9" width="0.1524" layer="16"/>
+<wire x1="37.8" y1="42.9" x2="41.2" y2="46.3" width="0.1524" layer="16"/>
+<via x="41.2" y="46.3" extent="1-16" drill="0.35"/>
+<wire x1="35.18" y1="46.3" x2="41.2" y2="46.3" width="0.1524" layer="16"/>
+<wire x1="32.21" y1="49.27" x2="35.18" y2="46.3" width="0.1524" layer="16"/>
 </signal>
 <signal name="N$16">
@@
 <wire x1="85.575" y1="17.825" x2="81.1" y2="22.3" width="0.1524" layer="1"/>
 <wire x1="81.1" y1="22.3" x2="71.9" y2="22.3" width="0.1524" layer="1"/>
-<wire x1="44.75" y1="44.83" x2="44.75" y2="45.85" width="0.1524" layer="16"/>
-<wire x1="43.5" y1="47.1" x2="41.2" y2="47.1" width="0.1524" layer="16"/>
-<wire x1="41.2" y1="47.1" x2="39.83" y2="48.47" width="0.1524" layer="16"/>
-<wire x1="39.83" y1="48.47" x2="39.83" y2="49.27" width="0.1524" layer="16"/>
-<wire x1="44.75" y1="45.85" x2="43.5" y2="47.1" width="0.1524" layer="16"/>
+<wire x1="39.83" y1="49.27" x2="39.83" y2="48.87" width="0.1524" layer="16"/>
+<wire x1="44.75" y1="44.83" x2="43.87" y2="44.83" width="0.1524" layer="16"/>
+<wire x1="43.87" y1="44.83" x2="39.83" y2="48.87" width="0.1524" layer="16"/>
 </signal>
 <signal name="RX_CAN1">
